Commit message: fix urdf & navigation

File: src/robot_simulation/urdf/robot_core.xacro (robot description, xacro)
@@ -1,180 +1,123 @@
 <?xml version="1.0"?>
-<robot xmlns:xacro="http://www.ros.org/wiki/xacro" name="diff_robot">
-  <!-- ======= Parameters ======= -->
-  <xacro:property name="robot_length" value="0.25"/>
-  <xacro:property name="robot_width"  value="0.25"/>
-  <xacro:property name="robot_height" value="0.10"/>
-  <xacro:property name="wheel_radius" value="0.035"/>
-  <xacro:property name="wheel_width"  value="0.03"/>
-  <xacro:property name="caster_radius" value="0.02"/>
-  <!-- ======= Base Link ======= -->
-  <link name="base_link">
-    <visual>
-      <geometry>
-        <box size="${robot_length} ${robot_width} ${robot_height}"/>
-      </geometry>
-      <origin xyz="0 0 ${robot_height/2}" rpy="0 0 0"/>
-      <material name="blue">
-        <color rgba="0.0 0.3 0.8 1.0"/>
-      </material>
-    </visual>
-    <collision>
-      <geometry>
-        <box size="${robot_length} ${robot_width} ${robot_height}"/>
-      </geometry>
-      <origin xyz="0 0 ${robot_height/2}" rpy="0 0 0"/>
-    </collision>
-    <inertial>
-      <mass value="4"/>
-      <origin xyz="0 0 ${robot_height/2}"/>
-      <inertia
-          ixx="0.02" ixy="0.0"  ixz="0.0"
-          iyy="0.04" iyz="0.0"
-          izz="0.05"/>
-    </inertial>
-  </link>
-  <!-- ============================
-       LEFT WHEEL
-  ============================= -->
-  <link name="left_wheel_link">
-    <visual>
-      <geometry>
-        <cylinder length="${wheel_width}" radius="${wheel_radius}"/>
-      </geometry>
-      <origin xyz="0 ${wheel_width/2} 0" rpy="1.5707 0 0"/>
-      <material name="black">
+<robot xmlns:xacro="http://www.ros.org/wiki/xacro" >
+    <!-- ======= Parameters ======= -->
+    <xacro:property name="chassis_length" value="0.335"/>
+    <xacro:property name="chassis_width" value="0.265"/>
+    <xacro:property name="chassis_height" value="0.138"/>
+    <xacro:property name="chassis_mass" value="1.0"/>
+    <xacro:property name="wheel_radius" value="0.033"/>
+    <xacro:property name="wheel_thickness" value="0.026"/>
+    <xacro:property name="wheel_mass" value="0.05"/>
+    <xacro:property name="wheel_offset_x" value="0.226"/>
+    <xacro:property name="wheel_offset_y" value="0.1485"/>
+    <xacro:property name="wheel_offset_z" value="0.01"/>
+    <xacro:property name="caster_wheel_radius" value="0.01"/>
+    <xacro:property name="caster_wheel_mass" value="2"/>
+    <xacro:property name="caster_wheel_offset_x" value="0.075"/>
+    <xacro:property name="caster_wheel_offset_z" value="${wheel_offset_z - wheel_radius + caster_wheel_radius}"/>
+    <material name="white">
+        <color rgba="1 1 1 1" />
+    </material>
+    <material name="orange">
+        <color rgba="1 0.3 0.1 1"/>
+    </material>
+    <material name="blue">
+        <color rgba="0.2 0.2 1 1"/>
+    </material>
+    <material name="black">
         <color rgba="0 0 0 1"/>
-      </material>
-    </visual>
-    <collision>
-      <geometry>
-        <cylinder length="${wheel_width}" radius="${wheel_radius}"/>
-      </geometry>
-      <origin xyz="0 ${wheel_width/2} 0" rpy="1.5707 0 0"/>
-    </collision>
-    <inertial>
-      <mass value="0.2"/>
-      <inertia ixx="0.001" ixy="0" ixz="0" iyy="0.001" iyz="0" izz="0.001"/>
-    </inertial>
-  </link>
-  <joint name="left_wheel_joint" type="continuous">
-    <parent link="base_link"/>
-    <child link="left_wheel_link"/>
-    <origin xyz="0 ${robot_width/2} 0" rpy="0 0 0"/>
-    <axis xyz="0 1 0"/>
-  </joint>
-  <!-- ============================
-       RIGHT WHEEL
-  ============================= -->
-  <link name="right_wheel_link">
-    <visual>
-      <geometry>
-        <cylinder length="${wheel_width}" radius="${wheel_radius}"/>
-      </geometry>
-      <origin xyz="0 -${wheel_width/2} 0" rpy="1.5707 0 0"/>
-      <material name="black">
-        <color rgba="0 0 0 1"/>
-      </material>
-    </visual>
-    <collision>
-      <geometry>
-        <cylinder length="${wheel_width}" radius="${wheel_radius}"/>
-      </geometry>
-      <origin xyz="0 -${wheel_width/2} 0" rpy="1.5707 0 0"/>
-    </collision>
-    <inertial>
-      <mass value="0.2"/>
-      <inertia ixx="0.001" ixy="0" ixz="0" iyy="0.001" iyz="0" izz="0.001"/>
-    </inertial>
-  </link>
-  <joint name="right_wheel_joint" type="continuous">
-    <parent link="base_link"/>
-    <child link="right_wheel_link"/>
-    <origin xyz="0 -${robot_width/2} 0" rpy="0 0 0"/>
-    <axis xyz="0 1 0"/>
-  </joint>
-  <!-- ============================
-       FRONT CASTER
-  ============================= -->
-  <link name="front_caster_link">
-    <visual>
-      <geometry>
-        <sphere radius="${caster_radius}"/>
-      </geometry>
-      <origin xyz="0 0 0" />
-      <material name="grey">
-        <color rgba="0.5 0.5 0.5 1"/>
-      </material>
-    </visual>
-    <collision>
-      <geometry><sphere radius="${caster_radius}"/></geometry>
-      <origin xyz="0 0 0"/>
-    </collision>
-  </link>
-  <joint name="front_caster_joint" type="fixed">
-    <parent link="base_link"/>
-    <child link="front_caster_link"/>
-    <origin xyz="${robot_length/2 - 0.03} 0 -0.015"/>
-  </joint>
-  <!-- ============================
-       REAR CASTER
-  ============================= -->
-  <link name="rear_caster_link">
-    <visual>
-      <geometry>
-        <sphere radius="${caster_radius}"/>
-      </geometry>
-      <origin xyz="-0 0 0" />
-      <material name="grey">
-        <color rgba="0.5 0.5 0.5 1"/>
-      </material>
-    </visual>
-    <collision>
-      <geometry><sphere radius="${caster_radius}"/></geometry>
-      <origin xyz="-0 0 0"/>
-    </collision>
-  </link>
-  <joint name="rear_caster_joint" type="fixed">
-    <parent link="base_link"/>
-    <child link="rear_caster_link"/>
-    <origin xyz="-${robot_length/2 - 0.03} 0 -0.015"/>
-  </joint>
-  <!-- ============================
-       LiDAR
-  ============================= -->
-  <link name="lidar_link">
-    <visual>
-      <geometry>
-        <cylinder length="0.03" radius="0.04"/>
-      </geometry>
-      <origin xyz="0 0 ${robot_height + 0.02}"/>
-      <material name="red">
+    </material>
+    <material name="red">
         <color rgba="1 0 0 1"/>
-      </material>
-    </visual>
-  </link>
-  <joint name="lidar_joint" type="fixed">
-    <parent link="base_link"/>
-    <child link="lidar_link"/>
-    <origin xyz="0 0 0"/>
-  </joint>
-  <!-- ============================
-       CAMERA (đã đổi tên)
-  ============================= -->
-  <link name="camera_front_link">
-    <visual>
-      <geometry>
-        <box size="0.05 0.05 0.03"/>
-      </geometry>
-      <origin xyz="0 0 0" />
-      <material name="green">
-        <color rgba="0 1 0 1"/>
-      </material>
-    </visual>
-  </link>
-  <joint name="camera_front_joint" type="fixed">
-    <parent link="base_link"/>
-    <child link="camera_front_link"/>
-    <origin xyz="${robot_length/2} 0 ${robot_height}"/>
-  </joint>
+    </material>
+    <!-- BASE LINK -->
+    <link name="base_link">
+    </link>
+    <!-- CHASSIS LINK -->
+    <joint name="chassis_joint" type="fixed">
+        <parent link="base_link"/>
+        <child link="chassis"/>
+        <origin xyz="${-wheel_offset_x} 0 ${-wheel_offset_z}"/>
+    </joint>
+    <link name="chassis">
+        <visual>
+            <origin xyz="${chassis_length/2} 0 ${chassis_height/2}"/>
+            <geometry>
+                <box size="${chassis_length} ${chassis_width} ${chassis_height}"/>
+            </geometry>
+            <material name="orange"/>
+        </visual>
+    </link>
+    <gazebo reference="chassis">
+        <material>Gazebo/Orange</material>
+    </gazebo>
+    <!-- LEFT WHEEL LINK -->
+    <joint name="left_wheel_joint" type="continuous">
+        <parent link="base_link"/>
+        <child link="left_wheel"/>
+        <origin xyz="0 ${wheel_offset_y} 0" rpy="-${pi/2} 0 0" />
+        <axis xyz="0 0 1"/>
+    </joint>
+    <link name="left_wheel">
+        <visual>
+            <geometry>
+                <cylinder radius="${wheel_radius}" length="${wheel_thickness}"/>
+            </geometry>
+            <material name="blue"/>
+        </visual>
+    </link>
+    <gazebo reference="left_wheel">
+        <material>Gazebo/Blue</material>
+    </gazebo>
+    <!-- RIGHT WHEEL LINK -->
+    <joint name="right_wheel_joint" type="continuous">
+        <parent link="base_link"/>
+        <child link="right_wheel"/>
+        <origin xyz="0 ${-wheel_offset_y} 0" rpy="${pi/2} 0 0" />
+        <axis xyz="0 0 -1"/>
+    </joint>
+    <link name="right_wheel">
+        <visual>
+            <geometry>
+                <cylinder radius="${wheel_radius}" length="${wheel_thickness}"/>
+            </geometry>
+            <material name="blue"/>
+        </visual>
+    </link>
+    <gazebo reference="right_wheel">
+        <material>Gazebo/Blue</material>
+    </gazebo>
+    <!-- CASTER WHEEL LINK -->
+    <joint name="caster_wheel_joint" type="fixed">
+        <parent link="chassis"/>
+        <child link="caster_wheel"/>
+        <origin xyz="${caster_wheel_offset_x} 0 ${caster_wheel_offset_z}"/>
+    </joint>
+    <link name="caster_wheel">
+        <visual>
+            <geometry>
+                <sphere radius="${caster_wheel_radius}"/>
+            </geometry>
+            <material name="white"/>
+        </visual>
+    </link>
+    <gazebo reference="caster_wheel">
+        <material>Gazebo/White</material>
+        <mu1 value="0.001"/>
+        <mu2 value="0.001"/>
+    </gazebo>
+    <!-- LASER-->
+    <joint name="laser_joint" type="fixed">
+        <parent link="base_link"/>
+        <child link="laser_frame"/>
+        <origin xyz="-0.1 0 0.175" rpy="0 0 3.14159"/>  <!--Điều chỉnh để cho phù hợp với chiều của lidar thực tế -->
+    </joint>
+    <link name="laser_frame">
+        <visual>
+            <geometry>
+                <cylinder radius="0.05" length="0.04"/>
+            </geometry>
+            <material name="red"/>
+        </visual>
+    </link>
 </robot>
